File: Nexus 01 schematic.kicad_sch (KiCad schematic)
At the start: 48 parts, among them J1 Conn_01x02_Male, J2 Conn_01x02_Male, J3 Conn_01x02_Male, J4 Conn_01x02_Male, J5 USB_C_Receptacle_USB2.0, J6 Conn_01x02_Male, Q1 SI2302, Q2 SI2302, Q3 SI2302, Q4 SI2302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

Commit message: Add files via upload
Parts:
- C1, C2, C4, C5, C6, C9: footprint (none) -> Capacitor_SMD:C_0603_1608Metric
- C3, C7, C8: footprint (none) -> Capacitor_SMD:C_0805_2012Metric
- D5, D6, D7: footprint (none) -> LED_SMD:LED_0603_1608Metric
- D8: footprint (none) -> Diode_SMD:D_SOD-323
- J1, J2, J3, J4, J6: footprint (none) -> Connector_PinHeader_1.00mm:PinHeader_1x02_P1.00mm_Vertical
- J5: footprint (none) -> Connector_USB:USB_C_Receptacle_HRO_TYPE-C-31-M-12; symbol Connector:USB_C_Receptacle_USB2.0 -> Connector:USB_C_Receptacle_USB2.0_16P
- R1, R10, R11, R12, R13, R14, R2, R3, R4, R5, R6, R7, R8, R9: footprint (none) -> Resistor_SMD:R_0603_1608Metric
- SW1, SW2: footprint (none) -> Button_Switch_SMD:SW_Push_1TS009xxxx-xxxx-xxxx_6x6x5mm
- U1: footprint (none) -> RF_Module:ESP32-S3-WROOM-1
